File: Hardware/avalon_communication_board.sch (KiCad schematic (older format))
At the start: 4 parts

Commit message: -Changed voltage regulator part to 12 - 3.3VDC Buck Converter -Updated voltage regulator schematic for new Buck Converter with new components as per datasheet
Parts:
- removed V1: LM2575D2T, symbol LM2575D2T
- added D1: 1N5820, symbol D_Schottky
- added V?: LM2576, symbol LM2576D2TR4-3.3G
- C2: value 330uF -> 1000uF
- L1: value 330uH -> 100uH
Connections:
- net labels added: +3.3V
- net labels removed: +5V
- wire segments 10 -> 12
Other:
- note added: "12 - 3.3VDC Regulator"
- note added: "Al"
- note removed: "12 - 5VDC Regulator"
- moved on the sheet: C1, C2, L1
Changed lines of the file:
@@
 LIBS:contrib
 LIBS:valves
+LIBS:avalon_communication_board-cache
 EELAYER 25 0
 EELAYER END
@@
 $EndDescr
 $Comp
-L LM2575D2T V1
-U 1 1 5A85BD4F
-P 2000 1350
-F 0 "V1" H 1800 1650 60  0000 C CNN
-F 1 "LM2575D2T" H 2000 1050 60  0000 C CNN
-F 2 "" H 2000 850 60  0000 C CNN
-F 3 "" H 2000 850 60  0000 C CNN
-	1    2000 1350
-	1    0    0    -1
-$EndComp
-$Comp
 L +12V #PWR?
 U 1 1 5A85BE6A
-P 1250 1000
-F 0 "#PWR?" H 1250 850 50  0001 C CNN
-F 1 "+12V" H 1250 1140 50  0000 C CNN
-F 2 "" H 1250 1000 50  0000 C CNN
-F 3 "" H 1250 1000 50  0000 C CNN
-	1    1250 1000
+P 800 850
+F 0 "#PWR?" H 800 700 50  0001 C CNN
+F 1 "+12V" H 800 990 50  0000 C CNN
+F 2 "" H 800 850 50  0000 C CNN
+F 3 "" H 800 850 50  0000 C CNN
+	1    800  850
 	1    0    0    -1
 $EndComp
 Wire Wire Line
-	1250 1200 1550 1200
+	800  1050 1100 1050
 $Comp
 L GND #PWR?
 U 1 1 5A85BEDF
-P 1250 1950
-F 0 "#PWR?" H 1250 1700 50  0001 C CNN
-F 1 "GND" H 1250 1800 50  0000 C CNN
-F 2 "" H 1250 1950 50  0000 C CNN
-F 3 "" H 1250 1950 50  0000 C CNN
-	1    1250 1950
+P 800 1800
+F 0 "#PWR?" H 800 1550 50  0001 C CNN
+F 1 "GND" H 800 1650 50  0000 C CNN
+F 2 "" H 800 1800 50  0000 C CNN
+F 3 "" H 800 1800 50  0000 C CNN
+	1    800  1800
 	1    0    0    -1
 $EndComp
@@
 L CP C1
 U 1 1 5A85BF83
-P 1250 1500
-F 0 "C1" H 1275 1600 50  0000 L CNN
-F 1 "100uF" H 1275 1400 50  0000 L CNN
-F 2 "" H 1288 1350 50  0000 C CNN
-F 3 "" H 1250 1500 50  0000 C CNN
-	1    1250 1500
+P 800 1350
+F 0 "C1" H 825 1450 50  0000 L CNN
+F 1 "100uF" H 825 1250 50  0000 L CNN
+F 2 "" H 838 1200 50  0000 C CNN
+F 3 "" H 800 1350 50  0000 C CNN
+	1    800  1350
 	1    0    0    -1
 $EndComp
 Wire Wire Line
-	1250 1000 1250 1350
-Connection ~ 1250 1200
+	800  850  800  1200
+Connection ~ 800  1050
 $Comp
 L INDUCTOR L1
 U 1 1 5A85C344
-P 2850 1500
-F 0 "L1" V 2800 1500 50  0000 C CNN
-F 1 "330uH" V 2950 1500 50  0000 C CNN
-F 2 "" H 2850 1500 50  0000 C CNN
-F 3 "" H 2850 1500 50  0000 C CNN
-	1    2850 1500
+P 2400 1350
+F 0 "L1" V 2350 1350 50  0000 C CNN
+F 1 "100uH" V 2500 1350 50  0000 C CNN
+F 2 "" H 2400 1350 50  0000 C CNN
+F 3 "" H 2400 1350 50  0000 C CNN
+	1    2400 1350
 	0    -1   -1   0
 $EndComp
 Wire Wire Line
-	3250 1200 2450 1200
+	2800 1050 2000 1050
 $Comp
 L CP C2
 U 1 1 5A85C5C7
-P 3250 1700
-F 0 "C2" H 3275 1800 50  0000 L CNN
-F 1 "330uF" H 3275 1600 50  0000 L CNN
-F 2 "" H 3288 1550 50  0000 C CNN
-F 3 "" H 3250 1700 50  0000 C CNN
-	1    3250 1700
+P 2800 1550
+F 0 "C2" H 2825 1650 50  0000 L CNN
+F 1 "1000uF" H 2825 1450 50  0000 L CNN
+F 2 "" H 2838 1400 50  0000 C CNN
+F 3 "" H 2800 1550 50  0000 C CNN
+	1    2800 1550
 	1    0    0    -1
 $EndComp
 Wire Wire Line
-	1550 1350 1550 1900
-Connection ~ 1550 1500
+	1100 1200 1100 1750
 Wire Wire Line
-	3150 1500 3800 1500
+	2700 1350 3350 1350
 Wire Wire Line
-	3250 1200 3250 1550
-Connection ~ 3250 1500
+	2800 1050 2800 1400
+Connection ~ 2800 1350
 Wire Wire Line
-	1250 1650 1250 1950
+	800  1500 800  1800
 Wire Wire Line
-	1250 1900 3250 1900
+	800  1750 2800 1750
 Wire Wire Line
-	3250 1900 3250 1850
-Connection ~ 1250 1900
-Connection ~ 1550 1900
+	2800 1750 2800 1700
+Connection ~ 800  1750
+Connection ~ 1100 1750
+Wire Wire Line
+	2100 1350 2000 1350
+Text Notes 1300 750  0    60   ~ 0
+12 - 3.3VDC Regulator
 $Comp
-L +5V #PWR?
-U 1 1 5A85CE89
-P 3800 1500
-F 0 "#PWR?" H 3800 1350 50  0001 C CNN
-F 1 "+5V" H 3800 1640 50  0000 C CNN
-F 2 "" H 3800 1500 50  0000 C CNN
-F 3 "" H 3800 1500 50  0000 C CNN
-	1    3800 1500
+L LM2576D2TR4-3.3G V?
+U 1 1 5A86207C
+P 1550 1200
+F 0 "V?" H 1350 1500 60  0000 C CNN
+F 1 "LM2576" H 1550 900 60  0000 C CNN
+F 2 "" H 1550 700 60  0000 C CNN
+F 3 "" H 1550 700 60  0000 C CNN
+	1    1550 1200
 	1    0    0    -1
 $EndComp
+Connection ~ 1100 1350
+$Comp
+L +3.3V #PWR?
+U 1 1 5A8624DD
+P 3350 1350
+F 0 "#PWR?" H 3350 1200 50  0001 C CNN
+F 1 "+3.3V" H 3350 1490 50  0000 C CNN
+F 2 "" H 3350 1350 50  0000 C CNN
+F 3 "" H 3350 1350 50  0000 C CNN
+	1    3350 1350
+	1    0    0    -1
+$EndComp
+Text Notes 600  1390 0    60   ~ 0
+Al
+$Comp
+L D_Schottky D1
+U 1 1 5A862E28
+P 2050 1550
+F 0 "D1" H 2050 1650 50  0000 C CNN
+F 1 "1N5820" H 2050 1450 50  0000 C CNN
+F 2 "" H 2050 1550 50  0000 C CNN
+F 3 "" H 2050 1550 50  0000 C CNN
+	1    2050 1550
+	0    1    1    0
+$EndComp
 Wire Wire Line
-	2550 1500 2450 1500
-Text Notes 1750 900  0    60   ~ 0
-12 - 5VDC Regulator
+	2050 1400 2050 1350
+Connection ~ 2050 1350
+Wire Wire Line
+	2050 1700 2050 1750
+Connection ~ 2050 1750
+Text Notes 2920 1590 0    60   ~ 0
+Al
 $EndSCHEMATC

Commit message: Started addition of Ultrasonic Transducer Control Circuitry
-Started schematic for H Bridge Circuit to drive Ultrasonic Transducer
Parts:
- added Q? (x2): BC817, symbol BC817
- added Q? (x2): FMMT597, symbol FMMT597
- added R? (x2): R, symbol R
- added U?: ultrasonic_transducer, symbol ultrasonic_transducer
Connections:
- wire segments 12 -> 21
Changed lines of the file:
@@
 Connection ~ 1100 1750
 Wire Wire Line
-	2100 1350 2000 1350
+	2000 1350 2100 1350
 Text Notes 1300 750  0    60   ~ 0
 12 - 3.3VDC Regulator
@@
 Text Notes 2920 1590 0    60   ~ 0
 Al
+$Comp
+L BC817 Q?
+U 1 1 5A8B3B7C
+P 2300 3950
+F 0 "Q?" H 2500 4000 50  0000 R CNN
+F 1 "BC817" H 2650 3900 50  0000 R CNN
+F 2 "" H 2400 4050 50  0000 C CNN
+F 3 "" H 2200 3950 50  0000 C CNN
+	1    2300 3950
+	1    0    0    -1
+$EndComp
+$Comp
+L BC817 Q?
+U 1 1 5A8B41ED
+P 3600 3000
+F 0 "Q?" H 3800 3050 50  0000 R CNN
+F 1 "BC817" H 3950 2950 50  0000 R CNN
+F 2 "" H 3700 3100 50  0000 C CNN
+F 3 "" H 3500 3000 50  0000 C CNN
+	1    3600 3000
+	-1   0    0    1
+$EndComp
+$Comp
+L FMMT597 Q?
+U 1 1 5A8B44D7
+P 3700 3950
+F 0 "Q?" H 4000 4000 50  0000 R CNN
+F 1 "FMMT597" H 4250 3900 50  0000 R CNN
+F 2 "" H 3900 4050 50  0000 C CNN
+F 3 "" H 3700 3950 50  0000 C CNN
+	1    3700 3950
+	-1   0    0    1
+$EndComp
+$Comp
+L FMMT597 Q?
+U 1 1 5A8B476E
+P 2200 3000
+F 0 "Q?" H 2500 3050 50  0000 R CNN
+F 1 "FMMT597" H 2750 2950 50  0000 R CNN
+F 2 "" H 2400 3100 50  0000 C CNN
+F 3 "" H 2200 3000 50  0000 C CNN
+	1    2200 3000
+	1    0    0    1
+$EndComp
+$Comp
+L ultrasonic_transducer U?
+U 1 1 5A8B4BD2
+P 2950 3450
+F 0 "U?" H 2950 3050 60  0000 C CNN
+F 1 "ultrasonic_transducer" H 2950 3150 60  0000 C CNN
+F 2 "" H 2950 3450 60  0000 C CNN
+F 3 "" H 2950 3450 60  0000 C CNN
+	1    2950 3450
+	1    0    0    -1
+$EndComp
+Wire Wire Line
+	3600 3200 3600 3750
+Wire Wire Line
+	3600 3450 3250 3450
+Connection ~ 3600 3450
+Wire Wire Line
+	2300 3200 2300 3750
+Wire Wire Line
+	2300 3450 2650 3450
+Connection ~ 2300 3450
+$Comp
+L R R?
+U 1 1 5A8B5409
+P 4150 3250
+F 0 "R?" V 4230 3250 50  0000 C CNN
+F 1 "R" V 4150 3250 50  0000 C CNN
+F 2 "" V 4080 3250 50  0000 C CNN
+F 3 "" H 4150 3250 50  0000 C CNN
+	1    4150 3250
+	1    0    0    -1
+$EndComp
+Wire Wire Line
+	3900 3000 4150 3000
+Wire Wire Line
+	4150 3000 4150 3100
+$Comp
+L R R?
+U 1 1 5A8B559E
+P 4150 3650
+F 0 "R?" V 4230 3650 50  0000 C CNN
+F 1 "R" V 4150 3650 50  0000 C CNN
+F 2 "" V 4080 3650 50  0000 C CNN
+F 3 "" H 4150 3650 50  0000 C CNN
+	1    4150 3650
+	1    0    0    -1
+$EndComp
+Wire Wire Line
+	4150 3950 3900 3950
+Wire Wire Line
+	4150 3800 4150 3950
+Wire Wire Line
+	4150 3400 4150 3500
 $EndSCHEMATC

Commit message: -Ultrasonic Transducer Driver Circuit completed
Parts:
- removed U?: ultrasonic_transducer, symbol ultrasonic_transducer
- added P1: B2P-VH, symbol B2P-VH
- added Q5: BC817, symbol BC817
- added R3, R6: 1K, symbol R
- added R4, R5: 1.5K, symbol R
- R1, R2: renamed from R?; value R -> 1.5K
- gave numbers to parts that had none: 5
Connections:
- net labels added: +5V, DUE144
- wire segments 21 -> 44
Other:
- note added: "PWM Pin 2"
- note added: "Ultrasonic Transducer Driver Circuit"
- moved on the sheet: Q1, Q2, Q3, Q4, R1, R2

Commit message: -Started production of Ethernet Controller Design -Updated Ultrasonic Transducer Driver Circuit to use 12V Supply instead of 5V Supply
Parts:
- added 400nF1: C, symbol C
- added IC1: ENC28J60-I/SO, SOIC-28, symbol ENC28J60-I/SO
- added J1: RJ45_LEDS, symbol RJ45_LEDS
- added R7, R8: 100R, symbol R
Connections:
- net labels added: LEDA, LEDB
- net labels removed: +5V
- wire segments 44 -> 71
Changed lines of the file:
@@
 Connection ~ 1400 3070
 $Comp
-L GND #PWR4
+L GND #PWR3
 U 1 1 5A8F5049
 P 2460 3910
-F 0 "#PWR4" H 2460 3660 50  0001 C CNN
+F 0 "#PWR3" H 2460 3660 50  0001 C CNN
 F 1 "GND" H 2460 3760 50  0000 C CNN
 F 2 "" H 2460 3910 50  0000 C CNN
@@
 	3100 3910 3100 3760
 Connection ~ 2460 3910
-$Comp
-L +5V #PWR3
-U 1 1 5A8F6ECD
-P 2380 2280
-F 0 "#PWR3" H 2380 2130 50  0001 C CNN
-F 1 "+5V" H 2380 2420 50  0000 C CNN
-F 2 "" H 2380 2280 50  0000 C CNN
-F 3 "" H 2380 2280 50  0000 C CNN
-	1    2380 2280
-	1    0    0    -1
-$EndComp
-Connection ~ 2380 2280
 Text GLabel 3930 4340 2    60   Input ~ 0
 DUE144
@@
 	0    1    1    0
 $EndComp
+$Comp
+L ENC28J60-I/SO IC1
+U 1 1 5A903E11
+P 7660 2460
+F 0 "IC1" H 7110 3410 50  0000 L CNN
+F 1 "ENC28J60-I/SO" H 7860 3410 50  0000 L CNN
+F 2 "SOIC-28" H 7660 2460 50  0000 C CIN
+F 3 "" H 7660 2460 50  0000 C CNN
+	1    7660 2460
+	1    0    0    -1
+$EndComp
+$Comp
+L RJ45_LEDS J1
+U 1 1 5A9063FA
+P 9910 2360
+F 0 "J1" H 9910 1860 50  0000 C CNN
+F 1 "RJ45_LEDS" H 9910 2760 50  0000 C CNN
+F 2 "" H 9910 2310 50  0000 C CNN
+F 3 "" H 9910 2310 50  0000 C CNN
+	1    9910 2360
+	0    1    1    0
+$EndComp
+$Comp
+L +12V #PWR4
+U 1 1 5A907F46
+P 2510 2280
+F 0 "#PWR4" H 2510 2130 50  0001 C CNN
+F 1 "+12V" H 2510 2420 50  0000 C CNN
+F 2 "" H 2510 2280 50  0000 C CNN
+F 3 "" H 2510 2280 50  0000 C CNN
+	1    2510 2280
+	1    0    0    -1
+$EndComp
+Connection ~ 2510 2280
+$Comp
+L +3.3V #PWR6
+U 1 1 5A908CDC
+P 7560 1090
+F 0 "#PWR6" H 7560 940 50  0001 C CNN
+F 1 "+3.3V" H 7560 1230 50  0000 C CNN
+F 2 "" H 7560 1090 50  0000 C CNN
+F 3 "" H 7560 1090 50  0000 C CNN
+	1    7560 1090
+	1    0    0    -1
+$EndComp
+Wire Wire Line
+	7560 1090 7560 1410
+Wire Wire Line
+	7760 1410 7760 1180
+Connection ~ 7560 1180
+Wire Wire Line
+	8360 1960 8620 1960
+Wire Wire Line
+	8620 1180 8620 2460
+Connection ~ 7760 1180
+Wire Wire Line
+	8620 2460 8360 2460
+Connection ~ 8620 1960
+$Comp
+L GND #PWR7
+U 1 1 5A90B1AB
+P 7560 3840
+F 0 "#PWR7" H 7560 3590 50  0001 C CNN
+F 1 "GND" H 7560 3690 50  0000 C CNN
+F 2 "" H 7560 3840 50  0000 C CNN
+F 3 "" H 7560 3840 50  0000 C CNN
+	1    7560 3840
+	1    0    0    -1
+$EndComp
+Wire Wire Line
+	7560 3510 7560 3840
+Wire Wire Line
+	7760 3510 7760 3740
+Wire Wire Line
+	8540 3740 7560 3740
+Connection ~ 7560 3740
+Wire Wire Line
+	8540 2260 8540 3740
+Wire Wire Line
+	8540 2760 8360 2760
+Connection ~ 7760 3740
+Wire Wire Line
+	8540 2260 8360 2260
+Connection ~ 8540 2760
+Wire Wire Line
+	7560 1180 8800 1180
+$Comp
+L C 400nF1
+U 1 1 5A90F1A9
+P 8950 1180
+F 0 "400nF1" H 8975 1280 50  0000 L CNN
+F 1 "C" H 8975 1080 50  0000 L CNN
+F 2 "" H 8988 1030 50  0000 C CNN
+F 3 "" H 8950 1180 50  0000 C CNN
+	1    8950 1180
+	0    -1   -1   0
+$EndComp
+Connection ~ 8620 1180
+$Comp
+L GND #PWR8
+U 1 1 5A90F671
+P 9240 1220
+F 0 "#PWR8" H 9240 970 50  0001 C CNN
+F 1 "GND" H 9240 1070 50  0000 C CNN
+F 2 "" H 9240 1220 50  0000 C CNN
+F 3 "" H 9240 1220 50  0000 C CNN
+	1    9240 1220
+	1    0    0    -1
+$EndComp
+Wire Wire Line
+	9100 1180 9240 1180
+Wire Wire Line
+	9240 1180 9240 1220
+Text GLabel 8810 1660 2    60   Input ~ 0
+LEDA
+Wire Wire Line
+	8360 1660 8810 1660
+Text GLabel 8810 1790 2    60   Input ~ 0
+LEDB
+Wire Wire Line
+	8360 1760 8680 1760
+Wire Wire Line
+	8680 1760 8680 1790
+Wire Wire Line
+	8680 1790 8810 1790
+$Comp
+L R R7
+U 1 1 5A911D20
+P 10650 2060
+F 0 "R7" V 10730 2060 50  0000 C CNN
+F 1 "100R" V 10650 2060 50  0000 C CNN
+F 2 "" V 10580 2060 50  0000 C CNN
+F 3 "" H 10650 2060 50  0000 C CNN
+	1    10650 2060
+	0    1    1    0
+$EndComp
+$Comp
+L R R8
+U 1 1 5A91211B
+P 10650 2760
+F 0 "R8" V 10730 2760 50  0000 C CNN
+F 1 "100R" V 10650 2760 50  0000 C CNN
+F 2 "" V 10580 2760 50  0000 C CNN
+F 3 "" H 10650 2760 50  0000 C CNN
+	1    10650 2760
+	0    1    1    0
+$EndComp
+Wire Wire Line
+	10410 2060 10500 2060
+Text GLabel 10880 1960 2    60   Input ~ 0
+LEDA
+Wire Wire Line
+	10410 1960 10880 1960
+$Comp
+L GND #PWR9
+U 1 1 5A913778
+P 11040 2400
+F 0 "#PWR9" H 11040 2150 50  0001 C CNN
+F 1 "GND" H 11040 2250 50  0000 C CNN
+F 2 "" H 11040 2400 50  0000 C CNN
+F 3 "" H 11040 2400 50  0000 C CNN
+	1    11040 2400
+	1    0    0    -1
+$EndComp
+Wire Wire Line
+	10800 2060 10920 2060
+Wire Wire Line
+	10920 2060 10920 2760
+Wire Wire Line
+	10920 2400 11040 2400
+Connection ~ 10920 2400
+Wire Wire Line
+	10920 2760 10800 2760
+Wire Wire Line
+	10500 2760 10410 2760
+Text GLabel 10660 2600 1    60   Input ~ 0
+LEDB
+Wire Wire Line
+	10410 2660 10660 2660
+Wire Wire Line
+	10660 2660 10660 2600
 $EndSCHEMATC
