File: Hardware/avalon_communication_board.sch (KiCad schematic (older format))
At the start: 41 parts, among them P1 B2P-VH, P10 8 Pin SIL, P11 8 Pin SIL, P2 MC34633, P3 MC34633, P4 MC34633, P5 MC34633, P6 6 Pin SIL, P7 10 Pin SIL, P8 8 Pin SIL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

Commit message: -Added camera transmission and switching electronics
-Added the camera switching chips from ROHM Semiconductor to enable
switching between 6 different video channels
-Added the camera transmission electronics taken from Blue Robotics
-Added 5V to -5V converter to drive camera transmission electronics
Parts:
- gave numbers to parts that had none: 1
Changed lines of the file:
@@
 EESchema Schematic File Version 2
-LIBS:avalon_communication_board-rescue
 LIBS:power
 LIBS:device
@@
 LIBS:contrib
 LIBS:valves
-LIBS:switches
 LIBS:avalon_communication_board-cache
 EELAYER 25 0
@@
 $EndDescr
 $Comp
-L +12V #PWR1
+L +12V #PWR01
 U 1 1 5A85BE6A
 P 800 850
-F 0 "#PWR1" H 800 700 50  0001 C CNN
+F 0 "#PWR01" H 800 700 50  0001 C CNN
 F 1 "+12V" H 800 990 50  0000 C CNN
 F 2 "" H 800 850 50  0000 C CNN
@@
 $EndComp
 $Comp
-L GND #PWR2
+L GND #PWR02
 U 1 1 5A85BEDF
 P 800 1800
-F 0 "#PWR2" H 800 1550 50  0001 C CNN
+F 0 "#PWR02" H 800 1550 50  0001 C CNN
 F 1 "GND" H 800 1650 50  0000 C CNN
 F 2 "" H 800 1800 50  0000 C CNN
@@
 $EndComp
 $Comp
-L +3.3V #PWR10
+L +3.3V #PWR03
 U 1 1 5A8624DD
 P 3350 1350
-F 0 "#PWR10" H 3350 1200 50  0001 C CNN
+F 0 "#PWR03" H 3350 1200 50  0001 C CNN
 F 1 "+3.3V" H 3350 1490 50  0000 C CNN
 F 2 "" H 3350 1350 50  0000 C CNN
@@
 $EndComp
 $Comp
-L GND #PWR5
+L GND #PWR04
 U 1 1 5A8F5049
 P 2460 3910
-F 0 "#PWR5" H 2460 3660 50  0001 C CNN
+F 0 "#PWR04" H 2460 3660 50  0001 C CNN
 F 1 "GND" H 2460 3760 50  0000 C CNN
 F 2 "" H 2460 3910 50  0000 C CNN
@@
 $EndComp
 $Comp
-L +12V #PWR6
+L +12V #PWR05
 U 1 1 5A907F46
 P 2510 2280
-F 0 "#PWR6" H 2510 2130 50  0001 C CNN
+F 0 "#PWR05" H 2510 2130 50  0001 C CNN
 F 1 "+12V" H 2510 2420 50  0000 C CNN
 F 2 "" H 2510 2280 50  0000 C CNN
@@
 $EndComp
 $Comp
-L +3.3V #PWR18
+L +3.3V #PWR06
 U 1 1 5A983E9A
 P 4255 6150
-F 0 "#PWR18" H 4255 6000 50  0001 C CNN
+F 0 "#PWR06" H 4255 6000 50  0001 C CNN
 F 1 "+3.3V" H 4255 6290 50  0000 C CNN
 F 2 "" H 4255 6150 50  0000 C CNN
@@
 $EndComp
 $Comp
-L GND #PWR12
+L GND #PWR07
 U 1 1 5A9843E8
 P 3525 6925
-F 0 "#PWR12" H 3525 6675 50  0001 C CNN
+F 0 "#PWR07" H 3525 6675 50  0001 C CNN
 F 1 "GND" H 3525 6775 50  0000 C CNN
 F 2 "" H 3525 6925 50  0000 C CNN
@@
 $EndComp
 $Comp
-L +3.3V #PWR3
+L +3.3V #PWR08
 U 1 1 5A98C3BB
 P 1270 6140
-F 0 "#PWR3" H 1270 5990 50  0001 C CNN
+F 0 "#PWR08" H 1270 5990 50  0001 C CNN
 F 1 "+3.3V" H 1270 6280 50  0000 C CNN
 F 2 "" H 1270 6140 50  0000 C CNN
@@
 $EndComp
 $Comp
-L GND #PWR4
+L GND #PWR09
 U 1 1 5A98C85B
 P 1275 6900
-F 0 "#PWR4" H 1275 6650 50  0001 C CNN
+F 0 "#PWR09" H 1275 6650 50  0001 C CNN
 F 1 "GND" H 1275 6750 50  0000 C CNN
 F 2 "" H 1275 6900 50  0000 C CNN
@@
 $EndComp
 $Comp
-L +12V #PWR13
+L +12V #PWR010
 U 1 1 5A9855AA
 P 3665 1010
-F 0 "#PWR13" H 3665 860 50  0001 C CNN
+F 0 "#PWR010" H 3665 860 50  0001 C CNN
 F 1 "+12V" H 3665 1150 50  0000 C CNN
 F 2 "" H 3665 1010 50  0000 C CNN
@@
 $EndComp
 $Comp
-L +5V #PWR22
+L +5V #PWR011
 U 1 1 5A989150
 P 5885 1180
-F 0 "#PWR22" H 5885 1030 50  0001 C CNN
+F 0 "#PWR011" H 5885 1030 50  0001 C CNN
 F 1 "+5V" H 5885 1320 50  0000 C CNN
 F 2 "" H 5885 1180 50  0000 C CNN
@@
 $EndComp
 $Comp
-L +5V #PWR20
+L +5V #PWR012
 U 1 1 5A9A1BCF
 P 5155 6145
-F 0 "#PWR20" H 5155 5995 50  0001 C CNN
+F 0 "#PWR012" H 5155 5995 50  0001 C CNN
 F 1 "+5V" H 5155 6285 50  0000 C CNN
 F 2 "" H 5155 6145 50  0000 C CNN
@@
 $EndComp
 $Comp
-L GND #PWR19
+L GND #PWR013
 U 1 1 5A9A225C
 P 5150 6720
-F 0 "#PWR19" H 5150 6470 50  0001 C CNN
+F 0 "#PWR013" H 5150 6470 50  0001 C CNN
 F 1 "GND" H 5150 6570 50  0000 C CNN
 F 2 "" H 5150 6720 50  0000 C CNN
@@
 $EndComp
 $Comp
-L +12V #PWR17
+L +12V #PWR014
 U 1 1 5A9A8159
 P 4025 5120
-F 0 "#PWR17" H 4025 4970 50  0001 C CNN
+F 0 "#PWR014" H 4025 4970 50  0001 C CNN
 F 1 "+12V" H 4025 5260 50  0000 C CNN
 F 2 "" H 4025 5120 50  0000 C CNN
@@
 $EndComp
 $Comp
-L +12V #PWR16
+L +12V #PWR015
 U 1 1 5A9A8E01
 P 3925 4940
-F 0 "#PWR16" H 3925 4790 50  0001 C CNN
+F 0 "#PWR015" H 3925 4790 50  0001 C CNN
 F 1 "+12V" H 3925 5080 50  0000 C CNN
 F 2 "" H 3925 4940 50  0000 C CNN
@@
 $EndComp
 $Comp
-L +5V #PWR15
+L +5V #PWR016
 U 1 1 5A9AD79D
 P 3825 5120
-F 0 "#PWR15" H 3825 4970 50  0001 C CNN
+F 0 "#PWR016" H 3825 4970 50  0001 C CNN
 F 1 "+5V" H 3825 5260 50  0000 C CNN
 F 2 "" H 3825 5120 50  0000 C CNN
@@
 $EndComp
 $Comp
-L +5V #PWR14
+L +5V #PWR017
 U 1 1 5A9AE118
 P 3725 5050
-F 0 "#PWR14" H 3725 4900 50  0001 C CNN
+F 0 "#PWR017" H 3725 4900 50  0001 C CNN
 F 1 "+5V" H 3725 5190 50  0000 C CNN
 F 2 "" H 3725 5050 50  0000 C CNN
@@
 $EndComp
 $Comp
-L +3.3V #PWR11
+L +3.3V #PWR018
 U 1 1 5A9B0550
 P 3485 5070
-F 0 "#PWR11" H 3485 4920 50  0001 C CNN
+F 0 "#PWR018" H 3485 4920 50  0001 C CNN
 F 1 "+3.3V" H 3485 5210 50  0000 C CNN
 F 2 "" H 3485 5070 50  0000 C CNN
@@
 $EndComp
 $Comp
-L +3.3V #PWR9
+L +3.3V #PWR019
 U 1 1 5A9B0BB3
 P 3325 5175
-F 0 "#PWR9" H 3325 5025 50  0001 C CNN
+F 0 "#PWR019" H 3325 5025 50  0001 C CNN
 F 1 "+3.3V" H 3325 5315 50  0000 C CNN
 F 2 "" H 3325 5175 50  0000 C CNN
@@
 $EndComp
 $Comp
-L GND #PWR8
+L GND #PWR020
 U 1 1 5A9B1CD1
 P 3200 4945
-F 0 "#PWR8" H 3200 4695 50  0001 C CNN
+F 0 "#PWR020" H 3200 4695 50  0001 C CNN
 F 1 "GND" H 3200 4795 50  0000 C CNN
 F 2 "" H 3200 4945 50  0000 C CNN
@@
 $EndComp
 $Comp
-L GND #PWR7
+L GND #PWR021
 U 1 1 5A9B23E5
 P 3100 5165
-F 0 "#PWR7" H 3100 4915 50  0001 C CNN
+F 0 "#PWR021" H 3100 4915 50  0001 C CNN
 F 1 "GND" H 3100 5015 50  0000 C CNN
 F 2 "" H 3100 5165 50  0000 C CNN
@@
 ULTRA_CTRL
 $Comp
-L +3.3V #PWR25
+L +3.3V #PWR022
 U 1 1 5A9E396C
 P 10635 4575
-F 0 "#PWR25" H 10635 4425 50  0001 C CNN
+F 0 "#PWR022" H 10635 4425 50  0001 C CNN
 F 1 "+3.3V" H 10635 4715 50  0000 C CNN
 F 2 "" H 10635 4575 50  0000 C CNN
@@
 $EndComp
 $Comp
-L GND #PWR24
+L GND #PWR023
 U 1 1 5A9E5137
 P 10515 4760
-F 0 "#PWR24" H 10515 4510 50  0001 C CNN
+F 0 "#PWR023" H 10515 4510 50  0001 C CNN
 F 1 "GND" H 10515 4610 50  0000 C CNN
 F 2 "" H 10515 4760 50  0000 C CNN
@@
 $EndComp
 $Comp
-L GND #PWR21
+L GND #PWR024
 U 1 1 5A999F70
 P 4670 4315
-F 0 "#PWR21" H 4670 4065 50  0001 C CNN
+F 0 "#PWR024" H 4670 4065 50  0001 C CNN
 F 1 "GND" H 4670 4165 50  0000 C CNN
 F 2 "" H 4670 4315 50  0000 C CNN
@@
 	4670 4200 4670 4315
 $Comp
-L +3.3V #PWR23
+L +3.3V #PWR025
 U 1 1 5A99EE06
 P 5595 2420
-F 0 "#PWR23" H 5595 2270 50  0001 C CNN
+F 0 "#PWR025" H 5595 2270 50  0001 C CNN
 F 1 "+3.3V" H 5595 2560 50  0000 C CNN
 F 2 "" H 5595 2420 50  0000 C CNN
@@
 	10440 2950 10500 2950
 $Comp
-L CONN_02X03 P?
+L CONN_02X03 P12
 U 1 1 5AA08E5D
 P 9555 1460
-F 0 "P?" H 9555 1660 50  0000 C CNN
+F 0 "P12" H 9555 1660 50  0000 C CNN
 F 1 "2x3 Pin SIL" H 9555 1260 50  0000 C CNN
 F 2 "" H 9555 260 50  0000 C CNN
