File: Hardware/ethernet_controller.sch (KiCad schematic (older format))
At the start: 20 parts

Commit message: -Continued work on the Ethernet Controller Schematic
Parts:
- 100mA: symbol Ferrite_Bead -> Ferrite_Bead-RESCUE-avalon_communication_board
- Y1: renamed from Y?; value Crystal -> ABM3-25MHz
- gave numbers to parts that had none: 16
- renumbered 100R to 100R1, 100R to 100R2
Connections:
- wire segments 137 -> 108
Other:
- moved on the sheet: C3
Changed lines of the file:
@@
 EESchema Schematic File Version 2
+LIBS:avalon_communication_board-rescue
 LIBS:power
 LIBS:device
@@
 $EndDescr
 $Comp
-L ENC28J60-I/SO IC?
+L ENC28J60-I/SO IC1
 U 1 1 5A920EF4
 P 3330 3255
-F 0 "IC?" H 2780 4205 50  0000 L CNN
+F 0 "IC1" H 2780 4205 50  0000 L CNN
 F 1 "ENC28J60-I/SO" H 3530 4205 50  0000 L CNN
 F 2 "SOIC-28" H 3330 3255 50  0000 C CIN
@@
 $EndComp
 $Comp
-L RJ45_LEDS J?
+L RJ45_LEDS J1
 U 1 1 5A920FD3
 P 7990 3135
-F 0 "J?" H 7990 2635 50  0000 C CNN
+F 0 "J1" H 7990 2635 50  0000 C CNN
 F 1 "RJ45_LEDS" H 7990 3535 50  0000 C CNN
 F 2 "" H 7990 3085 50  0000 C CNN
@@
 $EndComp
 $Comp
-L B78476A8247A003 U?
+L B78476A8247A003 U1
 U 1 1 5A9219B0
 P 6140 3085
-F 0 "U?" H 5840 3385 60  0000 C CNN
+F 0 "U1" H 5840 3385 60  0000 C CNN
 F 1 "B78476A8247A003" H 6140 2585 60  0000 C CNN
 F 2 "" H 6140 3085 60  0001 C CNN
@@
 $EndComp
 $Comp
-L +3.3V #PWR?
+L +3.3V #PWR6
 U 1 1 5A921B6A
 P 3230 1690
-F 0 "#PWR?" H 3230 1540 50  0001 C CNN
+F 0 "#PWR6" H 3230 1540 50  0001 C CNN
 F 1 "+3.3V" H 3230 1830 50  0000 C CNN
 F 2 "" H 3230 1690 50  0000 C CNN
@@
 LEDA
 $Comp
-L R 100R
+L R 100R1
 U 1 1 5A922478
 P 8695 2835
-F 0 "100R" V 8615 2835 50  0000 C CNN
+F 0 "100R1" V 8615 2835 50  0000 C CNN
 F 1 "R" V 8695 2835 50  0000 C CNN
 F 2 "" V 8625 2835 50  0000 C CNN
@@
 LEDB
 $Comp
-L R 100R
+L R 100R2
 U 1 1 5A922B30
 P 8730 3535
-F 0 "100R" V 8810 3535 50  0000 C CNN
+F 0 "100R2" V 8810 3535 50  0000 C CNN
 F 1 "R" V 8730 3535 50  0000 C CNN
 F 2 "" V 8660 3535 50  0000 C CNN
@@
 $EndComp
 $Comp
-L GND #PWR?
+L GND #PWR7
 U 1 1 5A92617F
 P 3230 4625
-F 0 "#PWR?" H 3230 4375 50  0001 C CNN
+F 0 "#PWR7" H 3230 4375 50  0001 C CNN
 F 1 "GND" H 3230 4475 50  0000 C CNN
 F 2 "" H 3230 4625 50  0000 C CNN
@@
 CAM2A
 $Comp
-L C C?
+L C C9
 U 1 1 5A92882C
 P 6850 3750
-F 0 "C?" H 6875 3850 50  0000 L CNN
+F 0 "C9" H 6875 3850 50  0000 L CNN
 F 1 "1nF" H 6875 3650 50  0000 L CNN
 F 2 "" H 6888 3600 50  0000 C CNN
@@
 $EndComp
 $Comp
-L R R?
+L R R11
 U 1 1 5A9159ED
 P 4815 2815
-F 0 "R?" V 4895 2815 50  0000 C CNN
+F 0 "R11" V 4895 2815 50  0000 C CNN
 F 1 "50R" V 4815 2815 50  0000 C CNN
 F 2 "" V 4745 2815 50  0000 C CNN
@@
 $EndComp
 $Comp
-L R R?
+L R R12
 U 1 1 5A915F14
 P 4815 3150
-F 0 "R?" V 4895 3150 50  0000 C CNN
+F 0 "R12" V 4895 3150 50  0000 C CNN
 F 1 "50R" V 4815 3150 50  0000 C CNN
 F 2 "" V 4745 3150 50  0000 C CNN
@@
 $EndComp
 $Comp
-L Ferrite_Bead 100mA
+L Ferrite_Bead-RESCUE-avalon_communication_board 100mA
 U 1 1 5A916F5B
 P 5060 2235
-F 0 "100mA" V 5010 2235 50  0000 C CNN
+AR Path="/5A916F5B" Ref="100mA"  Part="1"
+AR Path="/5A91950F/5A916F5B" Ref="100mA1"  Part="1"
+F 0 "100mA1" V 5010 2235 50  0000 C CNN
 F 1 "Ferrite_Bead" V 5160 2235 50  0000 C CNN
 F 2 "" H 5060 2235 50  0000 C CNN
@@
 $EndComp
 $Comp
-L C C?
+L C C8
 U 1 1 5A917819
 P 5060 3670
-F 0 "C?" H 5085 3770 50  0000 L CNN
+F 0 "C8" H 5085 3770 50  0000 L CNN
 F 1 "10nF" H 5085 3570 50  0000 L CNN
 F 2 "" H 5098 3520 50  0000 C CNN
@@
 $EndComp
 $Comp
-L R R?
+L R R9
 U 1 1 5A919DE1
 P 4560 3515
-F 0 "R?" V 4640 3515 50  0000 C CNN
+F 0 "R9" V 4640 3515 50  0000 C CNN
 F 1 "50R" V 4560 3515 50  0000 C CNN
 F 2 "" V 4490 3515 50  0000 C CNN
@@
 $EndComp
 $Comp
-L R R?
+L R R10
 U 1 1 5A919EB2
 P 4560 3890
-F 0 "R?" V 4640 3890 50  0000 C CNN
+F 0 "R10" V 4640 3890 50  0000 C CNN
 F 1 "50R" V 4560 3890 50  0000 C CNN
 F 2 "" V 4490 3890 50  0000 C CNN
@@
 $EndComp
 $Comp
-L C C?
+L C C7
 U 1 1 5A91B38D
 P 4785 4240
-F 0 "C?" H 4810 4340 50  0000 L CNN
+F 0 "C7" H 4810 4340 50  0000 L CNN
 F 1 "10nF" H 4810 4140 50  0000 L CNN
 F 2 "" H 4823 4090 50  0000 C CNN
@@
 $EndComp
 Wire Wire Line
-	3230 1690 3230 1740
-Wire Wire Line
-	3230 1740 3230 2205
+	3230 1690 3230 2205
 Wire Wire Line
 	3430 1740 3430 2205
 Wire Wire Line
-	2290 1740 2525 1740
-Wire Wire Line
-	2525 1740 3230 1740
-Wire Wire Line
-	3230 1740 3430 1740
-Wire Wire Line
-	3430 1740 3610 1740
-Wire Wire Line
-	3610 1740 4180 1740
-Wire Wire Line
-	4180 1740 5060 1740
+	2290 1740 5060 1740
 Connection ~ 3230 1740
 Wire Wire Line
@@
 	8490 3535 8580 3535
 Wire Wire Line
-	8880 4625 8880 3535
-Wire Wire Line
-	8880 3535 8880 2835
+	8880 4625 8880 2835
 Wire Wire Line
 	8880 2835 8845 2835
@@
 	4030 2755 4180 2755
 Wire Wire Line
-	4180 1740 4180 2755
-Wire Wire Line
-	4180 2755 4180 3255
+	4180 1740 4180 3255
 Connection ~ 3430 1740
 Wire Wire Line
@@
 	4030 3055 4115 3055
 Wire Wire Line
-	4115 4625 4115 3555
-Wire Wire Line
-	4115 3555 4115 3055
+	4115 3055 4115 4625
 Wire Wire Line
 	4115 3555 4030 3555
@@
 	3230 4625 3230 4305
 Wire Wire Line
-	1370 4625 2480 4625
-Wire Wire Line
-	2480 4625 3230 4625
-Wire Wire Line
-	3230 4625 3430 4625
-Wire Wire Line
-	3430 4625 4040 4625
-Wire Wire Line
-	4040 4625 4115 4625
-Wire Wire Line
-	4115 4625 4250 4625
-Wire Wire Line
-	4250 4625 4785 4625
-Wire Wire Line
-	4785 4625 5060 4625
-Wire Wire Line
-	5060 4625 6850 4625
-Wire Wire Line
-	6850 4625 8880 4625
+	1370 4625 8880 4625
 Connection ~ 4115 3555
 Wire Wire Line
@@
 	4490 2855 4490 2665
 Wire Wire Line
-	4490 2665 4815 2665
-Wire Wire Line
-	4815 2665 5540 2665
+	4490 2665 5540 2665
 Wire Wire Line
 	4030 2955 4490 2955
 Wire Wire Line
-	4490 3300 4815 3300
-Wire Wire Line
-	4815 3300 5365 3300
+	4490 3300 5365 3300
 Wire Wire Line
 	4490 2955 4490 3300
 Wire Wire Line
-	4815 2965 4815 2980
-Wire Wire Line
-	4815 2980 4815 3000
+	4815 2965 4815 3000
 Wire Wire Line
 	5365 3300 5365 3135
@@
 Connection ~ 4815 2665
 Wire Wire Line
-	4815 2980 5060 2980
-Wire Wire Line
-	5060 2980 5180 2980
-Wire Wire Line
-	5060 2535 5060 2980
-Wire Wire Line
-	5060 2980 5060 3520
+	4815 2980 5180 2980
+Wire Wire Line
+	5060 2535 5060 3520
 Connection ~ 4815 2980
 Connection ~ 4180 1740
@@
 	5060 3820 5060 4625
 Wire Wire Line
-	4030 3355 4560 3355
-Wire Wire Line
-	4560 3355 5435 3355
+	4030 3355 5435 3355
 Wire Wire Line
 	4560 3355 4560 3365
@@
 	4420 3455 4420 4040
 Wire Wire Line
-	4420 4040 4560 4040
-Wire Wire Line
-	4560 4040 5590 4040
-Wire Wire Line
-	4560 3665 4560 3715
-Wire Wire Line
-	4560 3715 4560 3740
+	4420 4040 5590 4040
+Wire Wire Line
+	4560 3665 4560 3740
 Wire Wire Line
 	5435 3355 5435 3235
@@
 	7205 3435 7205 3335
 $Comp
-L C C?
+L C C5
 U 1 1 5A9215F7
 P 3610 1930
-F 0 "C?" H 3635 2030 50  0000 L CNN
+F 0 "C5" H 3635 2030 50  0000 L CNN
 F 1 "400uF" H 3635 1830 50  0000 L CNN
 F 2 "" H 3648 1780 50  0000 C CNN
@@
 Connection ~ 3610 1740
 $Comp
-L GND #PWR?
+L GND #PWR8
 U 1 1 5A92196E
 P 3610 2080
-F 0 "#PWR?" H 3610 1830 50  0001 C CNN
+F 0 "#PWR8" H 3610 1830 50  0001 C CNN
 F 1 "GND" H 3610 1930 50  0000 C CNN
 F 2 "" H 3610 2080 50  0000 C CNN
@@
 $EndComp
 $Comp
-L R R?
+L R R7
 U 1 1 5A923613
 P 2525 2040
-F 0 "R?" V 2605 2040 50  0000 C CNN
+F 0 "R7" V 2605 2040 50  0000 C CNN
 F 1 "10K" V 2525 2040 50  0000 C CNN
 F 2 "" V 2455 2040 50  0000 C CNN
@@
 	2525 1890 2525 1740
 $Comp
-L C C?
+L C C6
 U 1 1 5A9244B5
 P 4250 4290
-F 0 "C?" H 4275 4390 50  0000 L CNN
+F 0 "C6" H 4275 4390 50  0000 L CNN
 F 1 "10uF" H 4275 4190 50  0000 L CNN
 F 2 "" H 4288 4140 50  0000 C CNN
@@
 $EndComp
 $Comp
-L R R?
+L R R8
 U 1 1 5A924614
 P 4040 4295
-F 0 "R?" V 3960 4295 50  0000 C CNN
+F 0 "R8" V 3960 4295 50  0000 C CNN
 F 1 "2K" V 4040 4295 50  0000 C CNN
 F 2 "" V 3970 4295 50  0000 C CNN
@@
 	2500 2955 2630 2955
 $Comp
-L Crystal Y?
+L Crystal Y1
 U 1 1 5A930E26
 P 2050 3700
-F 0 "Y?" H 2050 3850 50  0000 C CNN
-F 1 "Crystal" H 2050 3550 50  0000 C CNN
+F 0 "Y1" H 2050 3850 50  0000 C CNN
+F 1 "ABM3-25MHz" H 2050 3550 50  0000 C CNN
 F 2 "" H 2050 3700 50  0000 C CNN
 F 3 "" H 2050 3700 50  0000 C CNN
@@
 $EndComp
 $Comp
-L C C?
+L C C3
 U 1 1 5A9318BB
-P 1665 3450
-F 0 "C?" H 1690 3550 50  0000 L CNN
-F 1 "C" H 1690 3350 50  0000 L CNN
-F 2 "" H 1703 3300 50  0000 C CNN
-F 3 "" H 1665 3450 50  0000 C CNN
-	1    1665 3450
+P 1665 3330
+F 0 "C3" H 1690 3430 50  0000 L CNN
+F 1 "C" H 1690 3230 50  0000 L CNN
+F 2 "" H 1703 3180 50  0000 C CNN
+F 3 "" H 1665 3330 50  0000 C CNN
+	1    1665 3330
 	0    1    1    0
 $EndComp
 $Comp
-L C C?
+L C C4
 U 1 1 5A931944
 P 1670 3985
-F 0 "C?" H 1695 4085 50  0000 L CNN
+F 0 "C4" H 1695 4085 50  0000 L CNN
 F 1 "C" H 1695 3885 50  0000 L CNN
 F 2 "" H 1708 3835 50  0000 C CNN
@@
 $EndComp
 Wire Wire Line
-	1815 3450 2050 3450
-Wire Wire Line
-	2050 3450 2260 3450
-Wire Wire Line
-	1820 3985 2050 3985
-Wire Wire Line
-	2050 3985 2240 3985
-Wire Wire Line
-	2050 3450 2050 3550
+	1820 3985 2240 3985
+Wire Wire Line
+	2050 3330 2050 3550
 Wire Wire Line
 	2050 3985 2050 3850
 Wire Wire Line
-	2260 3450 2260 3555
-Wire Wire Line
-	2260 3555 2630 3555
-Connection ~ 2050 3450
+	2175 3555 2630 3555
 Wire Wire Line
 	2240 3985 2240 3755
@@
 Connection ~ 2050 3985
 Wire Wire Line
-	1515 3450 1370 3450
-Wire Wire Line
-	1370 3450 1370 3985
-Wire Wire Line
-	1370 3985 1370 4625
+	1370 3330 1370 4625
 Wire Wire Line
 	1370 3985 1520 3985
@@
 Text HLabel 2055 3025 0    60   Input ~ 0
 Ether_CS'
+Wire Wire Line
+	1370 3330 1515 3330
+Wire Wire Line
+	1815 3330 2175 3330
+Wire Wire Line
+	2175 3330 2175 3555
+Connection ~ 2050 3330
 $EndSCHEMATC

Commit message: -Ethernet controller schematic complete -Ferrite Bead component changed -Components selected and added to the communications board BOM, located in Google Drive -Filter Capacitor values changed to recommended values from Ethernet Controller datasheet
Parts:
- removed 100mA: Ferrite_Bead, symbol Ferrite_Bead-RESCUE-avalon_communication_board
- added C10, C11, C12: 0.1uF, symbol C
- added L2: Ferrite_Bead, symbol Ferrite_Bead
- C3, C4: value C -> 18pF
- C5: value 400uF -> 0.1uF
- R13: renamed from 100R1; value R -> 100R
- R14: renamed from 100R2; value R -> 100R
- R7: value 10K -> 100K
Connections:
- wire segments 108 -> 116
Changed lines of the file:
@@
 LEDA
 $Comp
-L R 100R1
+L R R13
 U 1 1 5A922478
 P 8695 2835
-F 0 "100R1" V 8615 2835 50  0000 C CNN
-F 1 "R" V 8695 2835 50  0000 C CNN
+F 0 "R13" V 8615 2835 50  0000 C CNN
+F 1 "100R" V 8695 2835 50  0000 C CNN
 F 2 "" V 8625 2835 50  0000 C CNN
 F 3 "" H 8695 2835 50  0000 C CNN
@@
 LEDB
 $Comp
-L R 100R2
+L R R14
 U 1 1 5A922B30
 P 8730 3535
-F 0 "100R2" V 8810 3535 50  0000 C CNN
-F 1 "R" V 8730 3535 50  0000 C CNN
+F 0 "R14" V 8810 3535 50  0000 C CNN
+F 1 "100R" V 8730 3535 50  0000 C CNN
 F 2 "" V 8660 3535 50  0000 C CNN
 F 3 "" H 8730 3535 50  0000 C CNN
@@
 L GND #PWR7
 U 1 1 5A92617F
-P 3230 4625
-F 0 "#PWR7" H 3230 4375 50  0001 C CNN
-F 1 "GND" H 3230 4475 50  0000 C CNN
-F 2 "" H 3230 4625 50  0000 C CNN
-F 3 "" H 3230 4625 50  0000 C CNN
-	1    3230 4625
+P 3230 4700
+F 0 "#PWR7" H 3230 4450 50  0001 C CNN
+F 1 "GND" H 3230 4550 50  0000 C CNN
+F 2 "" H 3230 4700 50  0000 C CNN
+F 3 "" H 3230 4700 50  0000 C CNN
+	1    3230 4700
 	1    0    0    -1
 $EndComp
@@
 $EndComp
 $Comp
-L Ferrite_Bead-RESCUE-avalon_communication_board 100mA
-U 1 1 5A916F5B
-P 5060 2235
-AR Path="/5A916F5B" Ref="100mA"  Part="1"
-AR Path="/5A91950F/5A916F5B" Ref="100mA1"  Part="1"
-F 0 "100mA1" V 5010 2235 50  0000 C CNN
-F 1 "Ferrite_Bead" V 5160 2235 50  0000 C CNN
-F 2 "" H 5060 2235 50  0000 C CNN
-F 3 "" H 5060 2235 50  0000 C CNN
-	1    5060 2235
-	1    0    0    -1
-$EndComp
-$Comp
 L C C8
 U 1 1 5A917819
@@
 	3430 1740 3430 2205
 Wire Wire Line
-	2290 1740 5060 1740
+	2290 1740 6585 1740
 Connection ~ 3230 1740
 Wire Wire Line
@@
 	4115 3555 4030 3555
 Wire Wire Line
-	3230 4625 3230 4305
+	3230 4305 3230 4700
 Wire Wire Line
 	1370 4625 8880 4625
@@
 	4815 2980 5180 2980
 Wire Wire Line
-	5060 2535 5060 3520
+	5060 2370 5060 3520
 Connection ~ 4815 2980
 Connection ~ 4180 1740
@@
 Connection ~ 5060 4625
 Wire Wire Line
-	5060 1740 5060 1935
+	5060 1740 5060 2070
 Wire Wire Line
 	5060 3820 5060 4625
@@
 Wire Wire Line
 	7205 3435 7205 3335
-$Comp
-L C C5
-U 1 1 5A9215F7
-P 3610 1930
-F 0 "C5" H 3635 2030 50  0000 L CNN
-F 1 "400uF" H 3635 1830 50  0000 L CNN
-F 2 "" H 3648 1780 50  0000 C CNN
-F 3 "" H 3610 1930 50  0000 C CNN
-	1    3610 1930
-	1    0    0    -1
-$EndComp
-Wire Wire Line
-	3610 1780 3610 1740
-Connection ~ 3610 1740
-$Comp
-L GND #PWR8
-U 1 1 5A92196E
-P 3610 2080
-F 0 "#PWR8" H 3610 1830 50  0001 C CNN
-F 1 "GND" H 3610 1930 50  0000 C CNN
-F 2 "" H 3610 2080 50  0000 C CNN
-F 3 "" H 3610 2080 50  0000 C CNN
-	1    3610 2080
-	1    0    0    -1
-$EndComp
 $Comp
 L R R7
@@
 P 2525 2040
 F 0 "R7" V 2605 2040 50  0000 C CNN
-F 1 "10K" V 2525 2040 50  0000 C CNN
+F 1 "100K" V 2525 2040 50  0000 C CNN
 F 2 "" V 2455 2040 50  0000 C CNN
 F 3 "" H 2525 2040 50  0000 C CNN
@@
 P 1665 3330
 F 0 "C3" H 1690 3430 50  0000 L CNN
-F 1 "C" H 1690 3230 50  0000 L CNN
+F 1 "18pF" H 1690 3230 50  0000 L CNN
 F 2 "" H 1703 3180 50  0000 C CNN
 F 3 "" H 1665 3330 50  0000 C CNN
@@
 P 1670 3985
 F 0 "C4" H 1695 4085 50  0000 L CNN
-F 1 "C" H 1695 3885 50  0000 L CNN
+F 1 "18pF" H 1695 3885 50  0000 L CNN
 F 2 "" H 1708 3835 50  0000 C CNN
 F 3 "" H 1670 3985 50  0000 C CNN
@@
 	2175 3330 2175 3555
 Connection ~ 2050 3330
+Wire Wire Line
+	5565 1740 5565 1810
+Connection ~ 5060 1740
+Wire Wire Line
+	5910 1740 5910 1810
+Connection ~ 5565 1740
+Wire Wire Line
+	6235 1740 6235 1810
+Connection ~ 5910 1740
+Wire Wire Line
+	6585 1740 6585 1810
+Connection ~ 6235 1740
+$Comp
+L GND #PWR8
+U 1 1 5A94B2CD
+P 6585 2205
+F 0 "#PWR8" H 6585 1955 50  0001 C CNN
+F 1 "GND" H 6585 2055 50  0000 C CNN
+F 2 "" H 6585 2205 50  0000 C CNN
+F 3 "" H 6585 2205 50  0000 C CNN
+	1    6585 2205
+	1    0    0    -1
+$EndComp
+Wire Wire Line
+	6585 2110 6585 2205
+Wire Wire Line
+	6235 2110 6235 2160
+Wire Wire Line
+	5565 2160 6585 2160
+Connection ~ 6585 2160
+Wire Wire Line
+	5910 2110 5910 2160
+Connection ~ 6235 2160
+Wire Wire Line
+	5565 2110 5565 2160
+Connection ~ 5910 2160
+$Comp
+L C C5
+U 1 1 5A95E0D5
+P 5565 1960
+F 0 "C5" H 5590 2060 50  0000 L CNN
+F 1 "0.1uF" H 5590 1860 50  0000 L CNN
+F 2 "" H 5603 1810 50  0000 C CNN
+F 3 "" H 5565 1960 50  0000 C CNN
+	1    5565 1960
+	1    0    0    -1
+$EndComp
+$Comp
+L C C10
+U 1 1 5A95E199
+P 5910 1960
+F 0 "C10" H 5935 2060 50  0000 L CNN
+F 1 "0.1uF" H 5935 1860 50  0000 L CNN
+F 2 "" H 5948 1810 50  0000 C CNN
+F 3 "" H 5910 1960 50  0000 C CNN
+	1    5910 1960
+	1    0    0    -1
+$EndComp
+$Comp
+L C C11
+U 1 1 5A95E20C
+P 6235 1960
+F 0 "C11" H 6260 2060 50  0000 L CNN
+F 1 "0.1uF" H 6260 1860 50  0000 L CNN
+F 2 "" H 6273 1810 50  0000 C CNN
+F 3 "" H 6235 1960 50  0000 C CNN
+	1    6235 1960
+	1    0    0    -1
+$EndComp
+$Comp
+L C C12
+U 1 1 5A95E276
+P 6585 1960
+F 0 "C12" H 6610 2060 50  0000 L CNN
+F 1 "0.1uF" H 6610 1860 50  0000 L CNN
+F 2 "" H 6623 1810 50  0000 C CNN
+F 3 "" H 6585 1960 50  0000 C CNN
+	1    6585 1960
+	1    0    0    -1
+$EndComp
+$Comp
+L Ferrite_Bead L2
+U 1 1 5A9617C1
+P 5060 2220
+F 0 "L2" V 4910 2245 50  0000 C CNN
+F 1 "Ferrite_Bead" V 5210 2220 50  0000 C CNN
+F 2 "" V 4990 2220 50  0000 C CNN
+F 3 "" H 5060 2220 50  0000 C CNN
+	1    5060 2220
+	1    0    0    -1
+$EndComp
 $EndSCHEMATC
